File: python/templates/template_with_symbols.kicad_sch (KiCad schematic)
At the start: 3 parts

Commit message: fix: update templates to KiCAD 9 format + remove corrupt _TEMPLATE_ blocks
Verified by live test: created a fresh schematic via MCP, result shows
format version 20250114, 0 _TEMPLATE_ hits, 0 (lib_id -100) hits, 24
real components placed cleanly.

--- Format version bump (20230121 KiCAD 7 -> 20250114 KiCAD 9) ---
Files: python/templates/*.kicad_sch, python/commands/project.py,
       python/commands/schematic.py

Root cause: the MCP server targets KiCAD 9 exclusively - pcbnew.pyd is
compiled for KiCAD 9.0 / Python 3.11.5, and server.ts explicitly selects
the KiCAD 9 bundled Python on Windows. Generating new schematics with a
2-year-old format tag caused a spurious 'This file was created with an
older KiCAD version' warning on every newly created schematic.

--- Remove corrupt _TEMPLATE_* placed-symbol blocks ---
File: python/templates/template_with_symbols_expanded.kicad_sch

Root cause: the expanded template was generated by the old sexpdata
serializer (same corruption PR #40 fixed for DynamicSymbolLoader add-path).
The serializer converted the string 'Device:R' to integer -100, producing
(lib_id -100) instead of (lib_id Device:R). KiCAD cannot resolve an
integer as a library reference and crashes with a null-pointer when the
user attempts to select these symbols. They appeared as grey _TEMPLATE_R?,
_TEMPLATE_C?, _TEMPLATE_U_REG? etc. ~5000mm off-sheet - invisible during
normal work but triggering a crash on accidental box-select.

Discovered via live testing on a real JLCPCB/KiCAD 9 project.
Connections:
- net at _TEMPLATE_R.1: now also _TEMPLATE_C.1
- net at _TEMPLATE_R.2: now also _TEMPLATE_C.2
Other:
- moved on the sheet: _TEMPLATE_C, _TEMPLATE_D, _TEMPLATE_R
Changed lines of the file:
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@@
-(kicad_sch (version 20230121) (generator "KiCAD-MCP-Server")
+(kicad_sch (version 20250114) (generator "KiCAD-MCP-Server")
   (paper "A4")
-  (symbol (lib_id "Device:R") (at -100 -100 0) (unit 1)
+  (symbol (lib_id "Device:R") (at -10000 -10000 0) (unit 1)
     (in_bom no) (on_board no) (dnp yes)
     (property "Reference" "_TEMPLATE_R" (at -100 -102.54 0)
@@
       (effects (font (size 1.27 1.27)) hide)
     )
-    (property "Datasheet" "~" (at -100 -100 0)
+    (property "Datasheet" "~" (at -10000 -10000 0)
       (effects (font (size 1.27 1.27)) hide)
     )
@@
     (pin "2")
   )
-  (symbol (lib_id "Device:C") (at -100 -110 0) (unit 1)
+  (symbol (lib_id "Device:C") (at -10000 -10000 0) (unit 1)
     (in_bom no) (on_board no) (dnp yes)
     (property "Reference" "_TEMPLATE_C" (at -100 -107.46 0)
@@
       (effects (font (size 1.27 1.27)))
     )
-    (property "Footprint" "" (at -100 -110 0)
+    (property "Footprint" "" (at -10000 -10000 0)
       (effects (font (size 1.27 1.27)) hide)
     )
-    (property "Datasheet" "~" (at -100 -110 0)
+    (property "Datasheet" "~" (at -10000 -10000 0)
       (effects (font (size 1.27 1.27)) hide)
     )
@@
     (pin "2")
   )
-  (symbol (lib_id "Device:LED") (at -100 -120 0) (unit 1)
+  (symbol (lib_id "Device:LED") (at -10000 -10000 0) (unit 1)
     (in_bom no) (on_board no) (dnp yes)
     (property "Reference" "_TEMPLATE_D" (at -100 -117.46 0)
@@
       (effects (font (size 1.27 1.27)))
     )
-    (property "Footprint" "" (at -100 -120 0)
+    (property "Footprint" "" (at -10000 -10000 0)
       (effects (font (size 1.27 1.27)) hide)
     )
-    (property "Datasheet" "~" (at -100 -120 0)
+    (property "Datasheet" "~" (at -10000 -10000 0)
       (effects (font (size 1.27 1.27)) hide)
     )
