File: python/templates/template_with_symbols_expanded.kicad_sch (KiCad schematic)
At the start: 13 parts

Commit message: fix: update templates to KiCAD 9 format + remove corrupt _TEMPLATE_ blocks
Verified by live test: created a fresh schematic via MCP, result shows
format version 20250114, 0 _TEMPLATE_ hits, 0 (lib_id -100) hits, 24
real components placed cleanly.

--- Format version bump (20230121 KiCAD 7 -> 20250114 KiCAD 9) ---
Files: python/templates/*.kicad_sch, python/commands/project.py,
       python/commands/schematic.py

Root cause: the MCP server targets KiCAD 9 exclusively - pcbnew.pyd is
compiled for KiCAD 9.0 / Python 3.11.5, and server.ts explicitly selects
the KiCAD 9 bundled Python on Windows. Generating new schematics with a
2-year-old format tag caused a spurious 'This file was created with an
older KiCAD version' warning on every newly created schematic.

--- Remove corrupt _TEMPLATE_* placed-symbol blocks ---
File: python/templates/template_with_symbols_expanded.kicad_sch

Root cause: the expanded template was generated by the old sexpdata
serializer (same corruption PR #40 fixed for DynamicSymbolLoader add-path).
The serializer converted the string 'Device:R' to integer -100, producing
(lib_id -100) instead of (lib_id Device:R). KiCAD cannot resolve an
integer as a library reference and crashes with a null-pointer when the
user attempts to select these symbols. They appeared as grey _TEMPLATE_R?,
_TEMPLATE_C?, _TEMPLATE_U_REG? etc. ~5000mm off-sheet - invisible during
normal work but triggering a crash on accidental box-select.

Discovered via live testing on a real JLCPCB/KiCAD 9 project.
Parts:
- removed _TEMPLATE_C: C, symbol Device:C
- removed _TEMPLATE_D: D, symbol Device:D
- removed _TEMPLATE_J2: Conn_2, symbol Connector_Generic:Conn_01x02
- removed _TEMPLATE_J4: Conn_4, symbol Connector_Generic:Conn_01x04
- removed _TEMPLATE_L: L, symbol Device:L
- removed _TEMPLATE_LED: LED, symbol Device:LED
- removed _TEMPLATE_Q_NMOS: Q_NMOS, symbol Device:Q_NMOS_GSD
- removed _TEMPLATE_Q_NPN: Q_NPN, symbol Device:Q_NPN_BCE
- removed _TEMPLATE_R: R, symbol Device:R
- removed _TEMPLATE_SW: Switch, symbol Switch:SW_Push
- removed _TEMPLATE_U_OPAMP: OpAmp, symbol Amplifier_Operational:LM358
- removed _TEMPLATE_U_REG: Regulator, symbol Regulator_Linear:AMS1117-3.3
- removed _TEMPLATE_Y: Crystal, symbol Device:Crystal
Changed lines of the file:
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@@
-(kicad_sch (version 20230121) (generator "KiCAD-MCP-Server")
+(kicad_sch (version 20250114) (generator "KiCAD-MCP-Server")
   (paper "A4")
-  ;; TEMPLATE INSTANCES (placed offscreen at -100, -110, etc.)
-  (symbol (lib_id "Device:R") (at -100 -100 0) (unit 1)
-    (in_bom no) (on_board no) (dnp yes)
-    (property "Reference" "_TEMPLATE_R" (at -100 -102.54 0)
-      (effects (font (size 1.27 1.27)))
-    )
-    (property "Value" "R" (at -100 -100 90)
-      (effects (font (size 1.27 1.27)))
-    )
-    (property "Footprint" "" (at -100 -100 90)
-      (effects (font (size 1.27 1.27)) hide)
-    )
-    (property "Datasheet" "~" (at -100 -100 0)
-      (effects (font (size 1.27 1.27)) hide)
-    )
-    (pin "1")
-    (pin "2")
-  )
-  (symbol (lib_id "Device:C") (at -100 -110 0) (unit 1)
-    (in_bom no) (on_board no) (dnp yes)
-    (property "Reference" "_TEMPLATE_C" (at -100 -107.46 0)
-      (effects (font (size 1.27 1.27)))
-    )
-    (property "Value" "C" (at -100 -112.54 0)
-      (effects (font (size 1.27 1.27)))
-    )
-    (property "Footprint" "" (at -100 -110 0)
-      (effects (font (size 1.27 1.27)) hide)
-    )
-    (property "Datasheet" "~" (at -100 -110 0)
-      (effects (font (size 1.27 1.27)) hide)
-    )
-    (pin "1")
-    (pin "2")
-  )
-  (symbol (lib_id "Device:L") (at -100 -120 0) (unit 1)
-    (in_bom no) (on_board no) (dnp yes)
-    (property "Reference" "_TEMPLATE_L" (at -100 -117.46 0)
-      (effects (font (size 1.27 1.27)))
-    )
-    (property "Value" "L" (at -100 -122.54 0)
-      (effects (font (size 1.27 1.27)))
-    )
-    (property "Footprint" "" (at -100 -120 0)
-      (effects (font (size 1.27 1.27)) hide)
-    )
-    (property "Datasheet" "~" (at -100 -120 0)
-      (effects (font (size 1.27 1.27)) hide)
-    )
-    (pin "1")
-    (pin "2")
-  )
-  (symbol (lib_id "Device:Crystal") (at -100 -130 0) (unit 1)
-    (in_bom no) (on_board no) (dnp yes)
-    (property "Reference" "_TEMPLATE_Y" (at -100 -127.46 0)
-      (effects (font (size 1.27 1.27)))
-    )
-    (property "Value" "Crystal" (at -100 -132.54 0)
-      (effects (font (size 1.27 1.27)))
-    )
-    (property "Footprint" "" (at -100 -130 0)
-      (effects (font (size 1.27 1.27)) hide)
-    )
-    (property "Datasheet" "~" (at -100 -130 0)
-      (effects (font (size 1.27 1.27)) hide)
-    )
-    (pin "1")
-    (pin "2")
-  )
-  (symbol (lib_id "Device:D") (at -100 -140 0) (unit 1)
-    (in_bom no) (on_board no) (dnp yes)
-    (property "Reference" "_TEMPLATE_D" (at -100 -137.46 0)
-      (effects (font (size 1.27 1.27)))
-    )
-    (property "Value" "D" (at -100 -142.54 0)
-      (effects (font (size 1.27 1.27)))
-    )
-    (property "Footprint" "" (at -100 -140 0)
-      (effects (font (size 1.27 1.27)) hide)
-    )
-    (property "Datasheet" "~" (at -100 -140 0)
-      (effects (font (size 1.27 1.27)) hide)
-    )
-    (pin "1")
-    (pin "2")
-  )
-  (symbol (lib_id "Device:LED") (at -100 -150 0) (unit 1)
-    (in_bom no) (on_board no) (dnp yes)
-    (property "Reference" "_TEMPLATE_LED" (at -100 -147.46 0)
-      (effects (font (size 1.27 1.27)))
-    )
-    (property "Value" "LED" (at -100 -152.54 0)
-      (effects (font (size 1.27 1.27)))
-    )
-    (property "Footprint" "" (at -100 -150 0)
-      (effects (font (size 1.27 1.27)) hide)
-    )
-    (property "Datasheet" "~" (at -100 -150 0)
-      (effects (font (size 1.27 1.27)) hide)
-    )
-    (pin "1")
-    (pin "2")
-  )
-  (symbol (lib_id "Device:Q_NPN_BCE") (at -100 -160 0) (unit 1)
-    (in_bom no) (on_board no) (dnp yes)
-    (property "Reference" "_TEMPLATE_Q_NPN" (at -100 -157.46 0)
-      (effects (font (size 1.27 1.27)))
-    )
-    (property "Value" "Q_NPN" (at -100 -162.54 0)
-      (effects (font (size 1.27 1.27)))
-    )
-    (property "Footprint" "" (at -100 -160 0)
-      (effects (font (size 1.27 1.27)) hide)
-    )
-    (property "Datasheet" "~" (at -100 -160 0)
-      (effects (font (size 1.27 1.27)) hide)
-    )
-    (pin "1")
-    (pin "2")
-    (pin "3")
-  )
-  (symbol (lib_id "Device:Q_NMOS_GSD") (at -100 -170 0) (unit 1)
-    (in_bom no) (on_board no) (dnp yes)
-    (property "Reference" "_TEMPLATE_Q_NMOS" (at -100 -167.46 0)
-      (effects (font (size 1.27 1.27)))
-    )
-    (property "Value" "Q_NMOS" (at -100 -172.54 0)
-      (effects (font (size 1.27 1.27)))
-    )
-    (property "Footprint" "" (at -100 -170 0)
-      (effects (font (size 1.27 1.27)) hide)
-    )
-    (property "Datasheet" "~" (at -100 -170 0)
-      (effects (font (size 1.27 1.27)) hide)
-    )
-    (pin "1")
-    (pin "2")
-    (pin "3")
-  )
-  (symbol (lib_id "Amplifier_Operational:LM358") (at -100 -180 0) (unit 1)
-    (in_bom no) (on_board no) (dnp yes)
-    (property "Reference" "_TEMPLATE_U_OPAMP" (at -100 -177.46 0)
-      (effects (font (size 1.27 1.27)))
-    )
-    (property "Value" "OpAmp" (at -100 -182.54 0)
-      (effects (font (size 1.27 1.27)))
-    )
-    (property "Footprint" "" (at -100 -180 0)
-      (effects (font (size 1.27 1.27)) hide)
-    )
-    (property "Datasheet" "" (at -100 -180 0)
-      (effects (font (size 1.27 1.27)) hide)
-    )
-    (pin "1")
-    (pin "2")
-    (pin "3")
-    (pin "4")
-    (pin "8")
-  )
-  (symbol (lib_id "Connector_Generic:Conn_01x02") (at -100 -190 0) (unit 1)
-    (in_bom no) (on_board no) (dnp yes)
-    (property "Reference" "_TEMPLATE_J2" (at -100 -187.46 0)
-      (effects (font (size 1.27 1.27)))
-    )
-    (property "Value" "Conn_2" (at -100 -192.54 0)
-      (effects (font (size 1.27 1.27)))
-    )
-    (property "Footprint" "" (at -100 -190 0)
-      (effects (font (size 1.27 1.27)) hide)
-    )
-    (property "Datasheet" "~" (at -100 -190 0)
-      (effects (font (size 1.27 1.27)) hide)
-    )
-    (pin "1")
-    (pin "2")
-  )
-  (symbol (lib_id "Connector_Generic:Conn_01x04") (at -100 -200 0) (unit 1)
-    (in_bom no) (on_board no) (dnp yes)
-    (property "Reference" "_TEMPLATE_J4" (at -100 -197.46 0)
-      (effects (font (size 1.27 1.27)))
-    )
-    (property "Value" "Conn_4" (at -100 -202.54 0)
-      (effects (font (size 1.27 1.27)))
-    )
-    (property "Footprint" "" (at -100 -200 0)
-      (effects (font (size 1.27 1.27)) hide)
-    )
-    (property "Datasheet" "~" (at -100 -200 0)
-      (effects (font (size 1.27 1.27)) hide)
-    )
-    (pin "1")
-    (pin "2")
-    (pin "3")
-    (pin "4")
-  )
-  (symbol (lib_id "Regulator_Linear:AMS1117-3.3") (at -100 -210 0) (unit 1)
-    (in_bom no) (on_board no) (dnp yes)
-    (property "Reference" "_TEMPLATE_U_REG" (at -100 -207.46 0)
-      (effects (font (size 1.27 1.27)))
-    )
-    (property "Value" "Regulator" (at -100 -212.54 0)
-      (effects (font (size 1.27 1.27)))
-    )
-    (property "Footprint" "" (at -100 -210 0)
-      (effects (font (size 1.27 1.27)) hide)
-    )
-    (property "Datasheet" "" (at -100 -210 0)
-      (effects (font (size 1.27 1.27)) hide)
-    )
-    (pin "1")
-    (pin "2")
-    (pin "3")
-  )
-  (symbol (lib_id "Switch:SW_Push") (at -100 -220 0) (unit 1)
-    (in_bom no) (on_board no) (dnp yes)
-    (property "Reference" "_TEMPLATE_SW" (at -100 -217.46 0)
-      (effects (font (size 1.27 1.27)))
-    )
-    (property "Value" "Switch" (at -100 -222.54 0)
-      (effects (font (size 1.27 1.27)))
-    )
-    (property "Footprint" "" (at -100 -220 0)
-      (effects (font (size 1.27 1.27)) hide)
-    )
-    (property "Datasheet" "~" (at -100 -220 0)
-      (effects (font (size 1.27 1.27)) hide)
-    )
-    (pin "1")
-    (pin "2")
-  )
   (sheet_instances
     (path "/" (page "1"))
